Commit message: added obj to urdf conversion, changes to spawn.py script and file structure in the project

File: resources/sample_urdf.urdf (robot description, URDF)
Before this commit: robot table.urdf, 1 links, 0 joints
Links:
- removed link baseLink
- added link , mass 1.0; collision mesh filename= scale=; visual mesh filename= scale=

Commit message: added obj to urdf conversion, changes to spawn.py script and file structure in the project

File: resources/sample_urdf.urdf (robot description, URDF)
Before this commit: robot table.urdf, 1 links, 0 joints
Links:
- removed link baseLink
- added link ; collision mesh filename= scale=; visual mesh filename= scale=
