Commit message: Kinect gravity

File: resources/cameras/kinect/kinect.urdf.xacro (robot description, xacro)
@@ -6,7 +6,10 @@
   <xacro:property name="mass" value="0.1" />
  <!-- Used for fixing robot to Gazebo 'base_link' -->
-  <link name="world"/>
+  <link name="kinect_world" />
+  <gazebo reference="kinect_world">
+    <gravity>0</gravity>
+  </gazebo>
   <joint name="fixed" type="fixed">
-    <parent link="world"/>
+    <parent link="kinect_world"/>
     <child link="kinect_link"/>
     <origin xyz="0 0 0.1" rpy="0 0 0"/>

Commit message: major overhaul of the project

File: resources/cameras/kinect/kinect.urdf.xacro (robot description, xacro)
@@ -17,10 +17,4 @@
   <!-- Kinect Link -->
   <link name="kinect_link">
-    <collision>
-      <origin xyz="0 0 0.1" rpy="0 0 0"/>
-      <geometry>
-          <mesh filename="package://image_generator/resources/cameras/kinect/kinect.dae" scale="0.001 0.001 0.001"/>
-      </geometry>
-    </collision>
     <visual>
       <origin xyz="0 0 0.1" rpy="0 0 0"/>

File: resources/sample_urdf.urdf (robot description, URDF)
Before this commit: robot , 1 links, 0 joints
Links:
- removed link 
- added link baseLink, mass 1; visual mesh filename= scale=
- added link gravity_link
Joints:
- added joint fixed: type fixed, parent gravity_link, child baseLink, origin xyz=0 0 0.1 rpy=0 0 0
